Commit message: [tb3_sim] depth camera added

File: sim/tb3_sim/urdf/turtlebot3_burger.urdf (robot description, URDF)
Before this commit: robot turtlebot3_burger, 12 links, 11 joints
Joints:
- joint camera_depth_joint: origin xyz=0.005 0.028 0.013 rpy=0 0 0 -> xyz=0.005 0.028 0.013 rpy=-1.57 0 -1.57
- joint camera_joint: origin xyz=0.064 0.0 0.24 rpy=0 0 0 -> xyz=-0.020 0.0 0.38 rpy=0 0 0
